File: HDTVii/HDTVii.sch (KiCad schematic (older format))
At the start: 27 parts

Commit message: forgotten to commit this idk
Parts:
- added C62, C79, C86: 50pF, symbol Device:C
- gave numbers to parts that had none: 1
Connections:
- net labels added: Unknown_Capacitance_Varistor_Replacements
Changed lines of the file:
@@
 F 2 "" H 7338 3500 50  0001 C CNN
 F 3 "~" H 7300 3650 50  0001 C CNN
-F 4 "6V" H 7182 3741 50  0000 R CNN "max. Voltage"
+F 4 "6V" H 7050 3750 50  0000 R CNN "max. Voltage"
 	1    7300 3650
 	-1   0    0    1
@@
 F 2 "" H 7988 3500 50  0001 C CNN
 F 3 "~" H 7950 3650 50  0001 C CNN
-F 4 "6V" H 7832 3741 50  0000 R CNN "max. Voltage"
+F 4 "6V" H 7700 3750 50  0000 R CNN "max. Voltage"
 	1    7950 3650
 	-1   0    0    1
@@
 F 2 "" H 6688 3500 50  0001 C CNN
 F 3 "~" H 6650 3650 50  0001 C CNN
-F 4 "6V" H 6532 3741 50  0000 R CNN "max. Voltage"
+F 4 "6V" H 6400 3750 50  0000 R CNN "max. Voltage"
 	1    6650 3650
 	-1   0    0    1
@@
 Connection ~ 4500 3950
 $Comp
-L Device:L FIL?
+L Device:L FIL15
 U 1 1 5ED97240
 P 5350 3800
-F 0 "FIL?" V 5450 3900 50  0000 R CNN
+F 0 "FIL15" V 5450 3900 50  0000 R CNN
 F 1 "280mH" V 5300 3950 50  0000 R CNN
 F 2 "" H 5350 3800 50  0001 C CNN
@@
 $EndComp
 Connection ~ 5350 3950
+$Comp
+L Device:C C86
+U 1 1 5ECD5101
+P 3850 5350
+F 0 "C86" V 3965 5396 50  0000 L CNN
+F 1 "50pF" H 3965 5305 50  0001 L CNN
+F 2 "" H 3888 5200 50  0001 C CNN
+F 3 "~" H 3850 5350 50  0001 C CNN
+	1    3850 5350
+	0    1    1    0
+$EndComp
+$Comp
+L Device:C C79
+U 1 1 5ECD5E01
+P 4700 5350
+F 0 "C79" V 4815 5396 50  0000 L CNN
+F 1 "50pF" H 4815 5305 50  0001 L CNN
+F 2 "" H 4738 5200 50  0001 C CNN
+F 3 "~" H 4700 5350 50  0001 C CNN
+	1    4700 5350
+	0    1    1    0
+$EndComp
+$Comp
+L Device:C C62
+U 1 1 5ECD629C
+P 5550 5350
+F 0 "C62" V 5665 5396 50  0000 L CNN
+F 1 "50pF" H 5665 5305 50  0001 L CNN
+F 2 "" H 5588 5200 50  0001 C CNN
+F 3 "~" H 5550 5350 50  0001 C CNN
+	1    5550 5350
+	0    1    1    0
+$EndComp
+Wire Notes Line
+	5900 6100 5900 5100
+Wire Notes Line
+	5900 5100 3500 5100
+Wire Notes Line
+	3500 5100 3500 6100
+Wire Notes Line
+	3500 6100 5900 6100
+Text GLabel 5550 5700 0    50   Input ~ 0
+Unknown_Capacitance_Varistor_Replacements
 Wire Bus Line
 	4300 2750 4300 4450

Commit message: Changed some stuff around I guess
Parts:
- removed W1, W2, W3, W4, W5, W6, W7, W8: Wire_Arc, symbol My~Library:Wire_Arc
- added W? (x8): Wire_Arc, symbol My_Library:Wire_Arc
- C64, C69, C84: value 220mF -> 220μF
- FIL15, FIL16, FIL17: value 280mH -> ?H
- W9: symbol My~Library:Wire_Arc -> My_Library:Wire_Arc
Connections:
- net labels removed: Unknown_Capacitance_Varistor_Replacements
Other:
- note added: "RVL-CPU-30 and earlier boards utilised capacitors\ninstead of the V1-V3 varistors. \nKnowing the value of either is trivial\nfor completing a safe replacemement\nof the component video circuitry."
- moved on the sheet: C62, C79, C86
