File: HDTVii/HDTVii.kicad_pcb (KiCad board)
At the start: 2 copper layers, 18 parts

Commit message: Changed many things
Parts:
- removed V1, V2, V3: Varistor, Resistor_SMD:R_0603_1608Metric_Pad1.05x0.95mm_HandSolder
- added D1: PESD5V0U1BA, Diode_SMD:D_SOD-323_HandSoldering, F.Cu at (201.4, 56.4)
- added D2: PESD5V0U1BA, Diode_SMD:D_SOD-323_HandSoldering, F.Cu at (201.4, 60.7)
- added D3: PESD5V0U1BA, Diode_SMD:D_SOD-323_HandSoldering, F.Cu at (203.7, 60.7)
- added D4: PESD5V0U1BA, Diode_SMD:D_SOD-323_HandSoldering, F.Cu at (206.0, 60.7)
- added J1: Conn_01x01_Male, Pad:pad, F.Cu at (203.7, 55.7)
- added J2: Conn_01x01_Male, Pad:pad, F.Cu at (206.4, 55.7)
- added J3: Conn_01x01_Male, Pad:pad, F.Cu at (209.1, 55.7)
- added J4: Conn_01x01_Male, Pad:pad, F.Cu at (211.3, 59.7)
- added J5: Conn_01x01_Male, Pad:pad, F.Cu at (211.8, 55.7)
- added J6: Conn_01x01_Male, Pad:pad, F.Cu at (211.3, 65.1)
- added J7: Conn_01x01_Male, Pad:pad, F.Cu at (211.3, 67.8)
- added J8: Conn_01x01_Male, Pad:pad, F.Cu at (211.3, 62.4)
- added J9: Conn_01x01_Male, Pad:pad, F.Cu at (206.4, 67.4)
- C64, C69, C84: footprint Capacitor_SMD:CP_Elec_6.3x3 -> Capacitor_Tantalum_SMD:CP_EIA-7343-15_Kemet-W_Pad2.25x2.55mm_HandSolder
- FIL15, FIL16, FIL17: value ?H -> 390nH
- moved FIL16 94.5 mm to (198.0, 57.6), turned to 180 degrees
- moved C74 92.7 mm to (198.0, 55.8), turned to 0 degrees
- moved FIL17 91.3 mm to (187.0, 57.6), turned to 180 degrees
- moved C78 90.0 mm to (195.4, 56.7), turned to 270 degrees
- moved C83 89.5 mm to (187.0, 55.8), turned to 0 degrees
- moved C85 86.7 mm to (184.4, 56.7), turned to 270 degrees
- moved FIL15 82.1 mm to (192.5, 57.6), turned to 180 degrees
- moved C66 80.4 mm to (192.5, 55.8), turned to 0 degrees
- moved C64 79.0 mm to (197.1, 63.8), turned to 90 degrees
- moved C72 77.5 mm to (189.9, 56.7), turned to 270 degrees
- moved C69 66.6 mm to (191.6, 63.8), turned to 90 degrees
- moved C84 55.2 mm to (186.1, 63.8), turned to 90 degrees
- moved R37 50.5 mm to (202.1, 63.9)
- moved R40 46.4 mm to (202.1, 65.8), turned to 180 degrees
- moved R39 43.2 mm to (202.1, 67.7), turned to 180 degrees
Connections:
- C69 pad 2: Net-(C69-Pad2) -> Net-(C66-Pad1)
- C72 pad 1: Net-(C72-Pad1) -> GND
- C74 pad 1: Net-(C74-Pad1) -> Net-(C64-Pad2)
- C78 pad 1: Net-(C78-Pad1) -> GND
- C78 pad 2: Net-(C74-Pad1) -> Net-(C64-Pad2)
- C84 pad 2: Net-(C84-Pad2) -> Net-(C83-Pad1)
- C85 pad 1: Net-(C85-Pad1) -> GND
- FIL16 pad 2: Net-(C74-Pad1) -> Net-(C64-Pad2)
- R37 pad 1: Net-(R37-Pad1) -> AVE54
- R37 pad 2: AVE59 -> GND
- R39 pad 1: AVE57 -> GND
- R39 pad 2: Net-(R39-Pad2) -> AVE57
- R40 pad 1: AVE54 -> GND
- R40 pad 2: Net-(R40-Pad2) -> AVE59
Routing:
- net AVE54: track 0.00 -> 27.1 mm
- net PrOut: track 0.00 -> 24.2 mm
- net AVE59: track 0.00 -> 21.1 mm
- net YOut: track 0.00 -> 18.4 mm
- net AVE57: track 0.00 -> 16.5 mm
- net MODE: track 0.00 -> 13.1 mm
- net PbOut: track 0.00 -> 12.0 mm
- net Net-(C66-Pad1): track 0.00 -> 7.48 mm
- net Net-(C83-Pad1): track 0.00 -> 7.38 mm
- net Net-(C64-Pad2): track 0.00 -> 7.32 mm
- net GND: vias 0 -> 11
- added copper zone on B.Cu, net GND
- added copper zone on F.Cu, net GND
Other:
- board outline added: 30 x 15 mm
- net class Default: clearance 0.2 -> 0.3; trace_width 0.25 -> 0.3
- rule trace_clearance: 0.2 -> 0.3
- board text added: "238"
- board text added: "54"
- board text added: "57"
- board text added: "59"
- board text added: "Job#3556 & Commandblock6417"
- board text added: "M"
- board text added: "Pb"
- board text added: "Pr"
- board text added: "Wii Component Video"
- board text added: "Y"
- board text added: "by"
