File: HDTVii/_saved_HDTVii.sch (KiCad schematic (older format))
At the start: 31 parts, among them J1 Conn_01x01_Male, J2 Conn_01x01_Male, J3 Conn_01x01_Male, J4 Conn_01x01_Male, J5 Conn_01x01_Male, J6 Conn_01x01_Male, J7 Conn_01x01_Male, J8 Conn_01x01_Male

Commit message: Changed many things
Parts:
- gave numbers to parts that had none: 1
Changed lines of the file:
@@
 	1500 3050 1150 3050
 $Comp
-L Connector:Conn_01x01_Male J?
+L Connector:Conn_01x01_Male J9
 U 1 1 5F07713C
 P 950 3600
-F 0 "J?" H 1056 3687 50  0001 C CNN
+F 0 "J9" H 1056 3687 50  0001 C CNN
 F 1 "Conn_01x01_Male" H 1056 3687 50  0001 C CNN
 F 2 "Pad:pad" H 950 3600 50  0001 C CNN
@@
 $EndComp
 $Comp
-L power:GND #PWR?
+L power:GND #PWR0111
 U 1 1 5F077E52
 P 1250 3700
-F 0 "#PWR?" H 1250 3450 50  0001 C CNN
+F 0 "#PWR0111" H 1250 3450 50  0001 C CNN
 F 1 "GND" H 1255 3527 50  0000 C CNN
 F 2 "" H 1250 3700 50  0001 C CNN
