File: miniRGBii/miniRGBii.sch (KiCad schematic (older format))
At the start: 28 parts

Commit message: Changed the board to utilise lower profile capacitors
Parts:
- C64, C69, C84: footprint Capacitor_Tantalum_SMD:CP_EIA-7343-15_Kemet-W_Pad2.25x2.55mm_HandSolder -> Capacitor_Tantalum_SMD:CP_EIA-6032-28_Kemet-C_Pad2.25x2.35mm_HandSolder
- FIL15, FIL16, FIL17: footprint Inductor_SMD:L_0402_1005Metric -> Inductor_SMD:L_0603_1608Metric_Pad1.05x0.95mm_HandSolder
Changed lines of the file:
@@
 F 0 "C64" H 5132 2659 50  0000 R CNN
 F 1 "220μF" H 5132 2750 50  0000 R CNN
-F 2 "Capacitor_Tantalum_SMD:CP_EIA-7343-15_Kemet-W_Pad2.25x2.55mm_HandSolder" H 5288 2600 50  0001 C CNN
+F 2 "Capacitor_Tantalum_SMD:CP_EIA-6032-28_Kemet-C_Pad2.25x2.35mm_HandSolder" H 5288 2600 50  0001 C CNN
 F 3 "~" H 5250 2750 50  0001 C CNN
 F 4 "6V" H 5000 2850 50  0000 R CNN "max. Voltage"
@@
 F 0 "C84" H 3832 2659 50  0000 R CNN
 F 1 "220μF" H 3832 2750 50  0000 R CNN
-F 2 "Capacitor_Tantalum_SMD:CP_EIA-7343-15_Kemet-W_Pad2.25x2.55mm_HandSolder" H 3988 2600 50  0001 C CNN
+F 2 "Capacitor_Tantalum_SMD:CP_EIA-6032-28_Kemet-C_Pad2.25x2.35mm_HandSolder" H 3988 2600 50  0001 C CNN
 F 3 "~" H 3950 2750 50  0001 C CNN
 F 4 "6V" H 3700 2850 50  0000 R CNN "max. Voltage"
@@
 F 0 "FIL17" V 4050 3750 50  0000 R CNN
 F 1 "390nH" V 3900 3750 50  0000 R CNN
-F 2 "Inductor_SMD:L_0402_1005Metric" H 3950 3650 50  0001 C CNN
+F 2 "Inductor_SMD:L_0603_1608Metric_Pad1.05x0.95mm_HandSolder" H 3950 3650 50  0001 C CNN
 F 3 "~" H 3950 3650 50  0001 C CNN
 	1    3950 3650
@@
 F 0 "FIL16" V 5350 3750 50  0000 R CNN
 F 1 "390nH" V 5200 3750 50  0000 R CNN
-F 2 "Inductor_SMD:L_0402_1005Metric" H 5250 3650 50  0001 C CNN
+F 2 "Inductor_SMD:L_0603_1608Metric_Pad1.05x0.95mm_HandSolder" H 5250 3650 50  0001 C CNN
 F 3 "~" H 5250 3650 50  0001 C CNN
 	1    5250 3650
@@
 F 0 "FIL15" V 6650 3750 50  0000 R CNN
 F 1 "390nH" V 6500 3750 50  0000 R CNN
-F 2 "Inductor_SMD:L_0402_1005Metric" H 6550 3650 50  0001 C CNN
+F 2 "Inductor_SMD:L_0603_1608Metric_Pad1.05x0.95mm_HandSolder" H 6550 3650 50  0001 C CNN
 F 3 "~" H 6550 3650 50  0001 C CNN
 	1    6550 3650
@@
 F 0 "C69" H 6432 2659 50  0000 R CNN
 F 1 "220μF" H 6432 2750 50  0000 R CNN
-F 2 "Capacitor_Tantalum_SMD:CP_EIA-7343-15_Kemet-W_Pad2.25x2.55mm_HandSolder" H 6588 2600 50  0001 C CNN
+F 2 "Capacitor_Tantalum_SMD:CP_EIA-6032-28_Kemet-C_Pad2.25x2.35mm_HandSolder" H 6588 2600 50  0001 C CNN
 F 3 "~" H 6550 2750 50  0001 C CNN
 F 4 "6V" H 6300 2850 50  0000 R CNN "max. Voltage"
