File: miniRGBii/miniRGBii.kicad_pcb (KiCad board)
At the start: 2 copper layers, 30 x 15 mm, 28 parts, among them J1 Conn_01x01_Male, J2 Conn_01x01_Male, J3 Conn_01x01_Male, J4 Conn_01x01_Male, J5 Conn_01x01_Male, J6 Conn_01x01_Male, J7 Conn_01x01_Male, J8 Conn_01x01_Male, J9 Conn_01x01_Male

Commit message: export to pdf, svg, gerber and more
Signed-off-by: Devnol <pgkoutsoumanis@gmail.com>
Other:
- rule pad_to_mask_clearance: 0.051 -> 0
Changed lines of the file:
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@@
   )
   (setup
-    (pad_to_mask_clearance 0.051)
-    (solder_mask_min_width 0.25)
+    (stackup
+      (layer "F.SilkS" (type "Top Silk Screen"))
+      (layer "F.Paste" (type "Top Solder Paste"))
+      (layer "F.Mask" (type "Top Solder Mask") (thickness 0.01))
+      (layer "F.Cu" (type "copper") (thickness 0.035))
+      (layer "dielectric 1" (type "core") (thickness 1.51) (material "FR4") (epsilon_r 4.5) (loss_tangent 0.02))
+      (layer "B.Cu" (type "copper") (thickness 0.035))
+      (layer "B.Mask" (type "Bottom Solder Mask") (thickness 0.01))
+      (layer "B.Paste" (type "Bottom Solder Paste"))
+      (layer "B.SilkS" (type "Bottom Silk Screen"))
+      (copper_finish "None")
+      (dielectric_constraints no)
+    )
+    (pad_to_mask_clearance 0)
     (pcbplotparams
-      (layerselection 0x00010f0_ffffffff)
+      (layerselection 0x00290f0_ffffffff)
       (disableapertmacros false)
       (usegerberextensions false)
@@
       (sketchpadsonfab false)
       (subtractmaskfromsilk false)
-      (outputformat 4)
+      (outputformat 1)
       (mirror false)
       (drillshape 0)
       (scaleselection 1)
-      (outputdirectory "images/output_layer_images_")
+      (outputdirectory "output_/")
     )
   )
@@
     (fp_line (start -3.65 -1.15) (end -3.65 2.15) (layer "F.Fab") (width 0.1))
     (fp_line (start 3.65 2.15) (end 3.65 -2.15) (layer "F.Fab") (width 0.1))
-    (pad "1" smd roundrect locked (at -3.2 0 90) (size 2.25 2.55) (layers "F.Cu" "F.Paste" "F.Mask") (roundrect_rratio 0.111111)
+    (pad "1" smd roundrect locked (at -3.2 0 90) (size 2.25 2.55) (layers "F.Cu" "F.Paste" "F.Mask") (roundrect_rratio 0.1111111111)
       (net 2 "AVE54") (pintype "passive"))
-    (pad "2" smd roundrect locked (at 3.2 0 90) (size 2.25 2.55) (layers "F.Cu" "F.Paste" "F.Mask") (roundrect_rratio 0.111111)
+    (pad "2" smd roundrect locked (at 3.2 0 90) (size 2.25 2.55) (layers "F.Cu" "F.Paste" "F.Mask") (roundrect_rratio 0.1111111111)
       (net 8 "Net-(C83-Pad1)") (pintype "passive"))
     (model "${KICAD6_3DMODEL_DIR}/Capacitor_Tantalum_SMD.3dshapes/CP_EIA-7343-15_Kemet-W.wrl"
@@
     (fp_line (start -3.65 -1.15) (end -3.65 2.15) (layer "F.Fab") (width 0.1))
     (fp_line (start 3.65 -2.15) (end -2.65 -2.15) (layer "F.Fab") (width 0.1))
-    (pad "1" smd roundrect locked (at -3.2 0 90) (size 2.25 2.55) (layers "F.Cu" "F.Paste" "F.Mask") (roundrect_rratio 0.111111)
+    (pad "1" smd roundrect locked (at -3.2 0 90) (size 2.25 2.55) (layers "F.Cu" "F.Paste" "F.Mask") (roundrect_rratio 0.1111111111)
       (net 4 "AVE59") (pintype "passive"))
-    (pad "2" smd roundrect locked (at 3.2 0 90) (size 2.25 2.55) (layers "F.Cu" "F.Paste" "F.Mask") (roundrect_rratio 0.111111)
+    (pad "2" smd roundrect locked (at 3.2 0 90) (size 2.25 2.55) (layers "F.Cu" "F.Paste" "F.Mask") (roundrect_rratio 0.1111111111)
       (net 7 "Net-(C66-Pad1)") (pintype "passive"))
     (model "${KICAD6_3DMODEL_DIR}/Capacitor_Tantalum_SMD.3dshapes/CP_EIA-7343-15_Kemet-W.wrl"
@@
     (fp_line (start 3.65 -2.15) (end -2.65 -2.15) (layer "F.Fab") (width 0.1))
     (fp_line (start -3.65 -1.15) (end -3.65 2.15) (layer "F.Fab") (width 0.1))
-    (pad "1" smd roundrect locked (at -3.2 0 90) (size 2.25 2.55) (layers "F.Cu" "F.Paste" "F.Mask") (roundrect_rratio 0.111111)
+    (pad "1" smd roundrect locked (at -3.2 0 90) (size 2.25 2.55) (layers "F.Cu" "F.Paste" "F.Mask") (roundrect_rratio 0.1111111111)
       (net 3 "AVE57") (pintype "passive"))
-    (pad "2" smd roundrect locked (at 3.2 0 90) (size 2.25 2.55) (layers "F.Cu" "F.Paste" "F.Mask") (roundrect_rratio 0.111111)
+    (pad "2" smd roundrect locked (at 3.2 0 90) (size 2.25 2.55) (layers "F.Cu" "F.Paste" "F.Mask") (roundrect_rratio 0.1111111111)
       (net 9 "Net-(C64-Pad2)") (pintype "passive"))
     (model "${KICAD6_3DMODEL_DIR}/Capacitor_Tantalum_SMD.3dshapes/CP_EIA-7343-15_Kemet-W.wrl"
@@
       (effects (font (size 1 1) (thickness 0.15)))
     )
-    (fp_text value "75Ω" (at 0 1.43 180) (layer "F.Fab")
+    (fp_text value "75Ω" (at 0 1.43 180) (layer "F.Fab") hide
       (effects (font (size 1 1) (thickness 0.15)))
     )
@@
       (effects (font (size 1 1) (thickness 0.15)))
     )
-    (fp_text value "75Ω" (at 0 1.43) (layer "F.Fab")
+    (fp_text value "75Ω" (at 0 1.43) (layer "F.Fab") hide
       (effects (font (size 1 1) (thickness 0.15)))
     )
@@
       (effects (font (size 1 1) (thickness 0.15)))
     )
-    (fp_text value "75Ω" (at 0 1.43 180) (layer "F.Fab")
+    (fp_text value "75Ω" (at 0 1.43 180) (layer "F.Fab") hide
       (effects (font (size 1 1) (thickness 0.15)))
     )
@@
   (zone (net 10) (net_name "GND") (layer "F.Cu") (hatch edge 0.508)
     (connect_pads thru_hole_only (clearance 0.3))
-    (min_thickness 0.3)
+    (min_thickness 0.3) (filled_areas_thickness no)
     (fill yes (thermal_gap 0.5) (thermal_bridge_width 0.5) (smoothing chamfer))
     (polygon
@@
   (zone (net 10) (net_name "GND") (layer "B.Cu") (hatch full 0.508)
     (connect_pads thru_hole_only (clearance 0.3))
-    (min_thickness 0.3)
+    (min_thickness 0.3) (filled_areas_thickness no)
     (fill yes (thermal_gap 0.5) (thermal_bridge_width 0.5))
     (polygon
@@
   (zone (net 0) (net_name "") (layer "B.Mask") (hatch edge 0.508)
     (connect_pads (clearance 0.3))
-    (min_thickness 0.254)
+    (min_thickness 0.254) (filled_areas_thickness no)
     (fill yes (thermal_gap 0.508) (thermal_bridge_width 0.508))
     (polygon
