File: miniRGBii_panel/miniRGBii.kicad_pcb (KiCad board)
At the start: 2 copper layers, 126 x 83 mm, 591 parts, among them J1 Conn_01x01_Male, J2 Conn_01x01_Male, J3 Conn_01x01_Male, J4 Conn_01x01_Male, J5 Conn_01x01_Male, J6 Conn_01x01_Male, J7 Conn_01x01_Male, J8 Conn_01x01_Male, J9 Conn_01x01_Male

Commit message: finalised (hopefully) the panel version
Parts:
- removed the C64 at (293.1, 131.8)
- removed the C64 at (261.1, 97.8)
- removed the C64 at (229.1, 97.8)
- removed the C64 at (197.1, 97.8)
- removed the C64 at (293.1, 80.8)
- removed the C64 at (261.1, 80.8)
- removed the C64 at (229.1, 80.8)
- removed the C64 at (197.1, 80.8)
- removed the C64 at (293.1, 63.8)
- removed the C64 at (261.1, 63.8)
- removed the C64 at (229.1, 63.8)
- removed the C64 at (261.1, 131.8)
- removed the C64 at (229.1, 131.8)
- removed the C64 at (197.1, 131.8)
- removed the C64 at (293.1, 114.8)
- removed the C64 at (261.1, 114.8)
- removed the C64 at (229.1, 114.8)
- removed the C64 at (197.1, 114.8)
- removed the C64 at (293.1, 97.8)
- removed the C66 at (288.5, 123.8)
- removed the C66 at (256.5, 89.8)
- removed the C66 at (224.5, 89.8)
- removed the C66 at (192.5, 89.8)
- removed the C66 at (288.5, 72.8)
- removed the C66 at (256.5, 72.8)
- removed the C66 at (224.5, 72.8)
- removed the C66 at (192.5, 72.8)
- removed the C66 at (288.5, 55.8)
- removed the C66 at (256.5, 55.8)
- removed the C66 at (224.5, 55.8)
- removed the C66 at (256.5, 123.8)
- removed the C66 at (224.5, 123.8)
- removed the C66 at (192.5, 123.8)
- removed the C66 at (288.5, 106.8)
- removed the C66 at (256.5, 106.8)
- removed the C66 at (224.5, 106.8)
- removed the C66 at (192.5, 106.8)
- removed the C66 at (288.5, 89.8)
- removed the C69 at (287.6, 131.8)
- removed the C69 at (255.6, 97.8)
- removed the C69 at (223.6, 97.8)
- removed the C69 at (191.6, 97.8)
- removed the C69 at (287.6, 80.8)
- removed the C69 at (255.6, 80.8)
- removed the C69 at (223.6, 80.8)
- removed the C69 at (191.6, 80.8)
- removed the C69 at (287.6, 63.8)
- removed the C69 at (255.6, 63.8)
- removed the C69 at (223.6, 63.8)
- removed the C69 at (255.6, 131.8)
- removed the C69 at (223.6, 131.8)
- removed the C69 at (191.6, 131.8)
- removed the C69 at (287.6, 114.8)
- removed the C69 at (255.6, 114.8)
- removed the C69 at (223.6, 114.8)
- removed the C69 at (191.6, 114.8)
- removed the C69 at (287.6, 97.8)
- removed the C72 at (285.9, 124.7)
- removed the C72 at (253.9, 90.7)
- removed the C72 at (221.9, 90.7)
- removed the C72 at (189.9, 90.7)
- removed the C72 at (285.9, 73.7)
- removed the C72 at (253.9, 73.7)
- removed the C72 at (221.9, 73.7)
- removed the C72 at (189.9, 73.7)
- removed the C72 at (285.9, 56.7)
- removed the C72 at (253.9, 56.7)
- removed the C72 at (221.9, 56.7)
- removed the C72 at (253.9, 124.7)
- removed the C72 at (221.9, 124.7)
- removed the C72 at (189.9, 124.7)
- removed the C72 at (285.9, 107.7)
- removed the C72 at (253.9, 107.7)
- removed the C72 at (221.9, 107.7)
- removed the C72 at (189.9, 107.7)
- removed the C72 at (285.9, 90.7)
- removed the C74 at (294.0, 123.8)
- removed the C74 at (262.0, 89.8)
- removed the C74 at (230.0, 89.8)
- removed the C74 at (198.0, 89.8)
- removed the C74 at (294.0, 72.8)
- removed the C74 at (262.0, 72.8)
- removed the C74 at (230.0, 72.8)
- removed the C74 at (198.0, 72.8)
- removed the C74 at (294.0, 55.8)
- removed the C74 at (262.0, 55.8)
- removed the C74 at (230.0, 55.8)
- removed the C74 at (262.0, 123.8)
- removed the C74 at (230.0, 123.8)
- removed the C74 at (198.0, 123.8)
- removed the C74 at (294.0, 106.8)
- removed the C74 at (262.0, 106.8)
- removed the C74 at (230.0, 106.8)
- removed the C74 at (198.0, 106.8)
- removed the C74 at (294.0, 89.8)
- removed the C78 at (291.4, 124.7)
- removed the C78 at (259.4, 90.7)
- removed the C78 at (227.4, 90.7)
- removed the C78 at (195.4, 90.7)
- removed the C78 at (291.4, 73.7)
- removed the C78 at (259.4, 73.7)
- removed the C78 at (227.4, 73.7)
- removed the C78 at (195.4, 73.7)
- removed the C78 at (291.4, 56.7)
- removed the C78 at (259.4, 56.7)
- removed the C78 at (227.4, 56.7)
- removed the C78 at (259.4, 124.7)
- removed the C78 at (227.4, 124.7)
- removed the C78 at (195.4, 124.7)
- removed the C78 at (291.4, 107.7)
- removed the C78 at (259.4, 107.7)
- removed the C78 at (227.4, 107.7)
- removed the C78 at (195.4, 107.7)
- removed the C78 at (291.4, 90.7)
- removed the C83 at (283.0, 123.8)
- removed the C83 at (251.0, 89.8)
- removed the C83 at (219.0, 89.8)
- removed the C83 at (187.0, 89.8)
- removed the C83 at (283.0, 72.8)
- removed the C83 at (251.0, 72.8)
- removed the C83 at (219.0, 72.8)
- removed the C83 at (187.0, 72.8)
- removed the C83 at (283.0, 55.8)
- removed the C83 at (251.0, 55.8)
- removed the C83 at (219.0, 55.8)
- removed the C83 at (251.0, 123.8)
- removed the C83 at (219.0, 123.8)
- removed the C83 at (187.0, 123.8)
- removed the C83 at (283.0, 106.8)
- removed the C83 at (251.0, 106.8)
- removed the C83 at (219.0, 106.8)
- removed the C83 at (187.0, 106.8)
- removed the C83 at (283.0, 89.8)
- removed the C84 at (282.1, 131.8)
- removed the C84 at (250.1, 97.8)
- removed the C84 at (218.1, 97.8)
- removed the C84 at (186.1, 97.8)
- removed the C84 at (282.1, 80.8)
- removed the C84 at (250.1, 80.8)
- removed the C84 at (218.1, 80.8)
- removed the C84 at (186.1, 80.8)
- removed the C84 at (282.1, 63.8)
- removed the C84 at (250.1, 63.8)
- removed the C84 at (218.1, 63.8)
- removed the C84 at (250.1, 131.8)
- removed the C84 at (218.1, 131.8)
- removed the C84 at (186.1, 131.8)
- removed the C84 at (282.1, 114.8)
- removed the C84 at (250.1, 114.8)
- removed the C84 at (218.1, 114.8)
- removed the C84 at (186.1, 114.8)
- removed the C84 at (282.1, 97.8)
- removed the C85 at (280.4, 124.7)
- removed the C85 at (248.4, 90.7)
- removed the C85 at (216.4, 90.7)
- removed the C85 at (184.4, 90.7)
- removed the C85 at (280.4, 73.7)
- removed the C85 at (248.4, 73.7)
- removed the C85 at (216.4, 73.7)
- removed the C85 at (184.4, 73.7)
- removed the C85 at (280.4, 56.7)
- removed the C85 at (248.4, 56.7)
- removed the C85 at (216.4, 56.7)
- removed the C85 at (248.4, 124.7)
- removed the C85 at (216.4, 124.7)
- removed the C85 at (184.4, 124.7)
- removed the C85 at (280.4, 107.7)
- removed the C85 at (248.4, 107.7)
- removed the C85 at (216.4, 107.7)
- removed the C85 at (184.4, 107.7)
- removed the C85 at (280.4, 90.7)
- removed the D1 at (297.4, 124.4)
- removed the D1 at (265.4, 90.4)
- removed the D1 at (233.4, 90.4)
- removed the D1 at (201.4, 90.4)
- removed the D1 at (297.4, 73.4)
- removed the D1 at (265.4, 73.4)
- removed the D1 at (233.4, 73.4)
- removed the D1 at (201.4, 73.4)
- removed the D1 at (297.4, 56.4)
- removed the D1 at (265.4, 56.4)
- removed the D1 at (233.4, 56.4)
- removed the D1 at (265.4, 124.4)
- removed the D1 at (233.4, 124.4)
- removed the D1 at (201.4, 124.4)
- removed the D1 at (297.4, 107.4)
- removed the D1 at (265.4, 107.4)
- removed the D1 at (233.4, 107.4)
- removed the D1 at (201.4, 107.4)
- removed the D1 at (297.4, 90.4)
- removed the D2 at (297.4, 128.7)
- removed the D2 at (265.4, 94.7)
- removed the D2 at (233.4, 94.7)
- removed the D2 at (201.4, 94.7)
- removed the D2 at (297.4, 77.7)
- removed the D2 at (265.4, 77.7)
- removed the D2 at (233.4, 77.7)
- removed the D2 at (201.4, 77.7)
- removed the D2 at (297.4, 60.7)
- removed the D2 at (265.4, 60.7)
- removed the D2 at (233.4, 60.7)
- removed the D2 at (265.4, 128.7)
- removed the D2 at (233.4, 128.7)
- removed the D2 at (201.4, 128.7)
- removed the D2 at (297.4, 111.7)
- removed the D2 at (265.4, 111.7)
- removed the D2 at (233.4, 111.7)
- removed the D2 at (201.4, 111.7)
- removed the D2 at (297.4, 94.7)
- removed the D3 at (299.7, 128.7)
- removed the D3 at (267.7, 94.7)
- removed the D3 at (235.7, 94.7)
- removed the D3 at (203.7, 94.7)
- removed the D3 at (299.7, 77.7)
- removed the D3 at (267.7, 77.7)
- removed the D3 at (235.7, 77.7)
- removed the D3 at (203.7, 77.7)
- removed the D3 at (299.7, 60.7)
- removed the D3 at (267.7, 60.7)
- removed the D3 at (235.7, 60.7)
- removed the D3 at (267.7, 128.7)
- removed the D3 at (235.7, 128.7)
- removed the D3 at (203.7, 128.7)
- removed the D3 at (299.7, 111.7)
- removed the D3 at (267.7, 111.7)
- removed the D3 at (235.7, 111.7)
- removed the D3 at (203.7, 111.7)
- removed the D3 at (299.7, 94.7)
- removed the D4 at (302.0, 128.7)
- removed the D4 at (270.0, 94.7)
- removed the D4 at (238.0, 94.7)
- removed the D4 at (206.0, 94.7)
- removed the D4 at (302.0, 77.7)
- removed the D4 at (270.0, 77.7)
- removed the D4 at (238.0, 77.7)
- removed the D4 at (206.0, 77.7)
- removed the D4 at (302.0, 60.7)
- removed the D4 at (270.0, 60.7)
- removed the D4 at (238.0, 60.7)
- removed the D4 at (270.0, 128.7)
- removed the D4 at (238.0, 128.7)
- removed the D4 at (206.0, 128.7)
- removed the D4 at (302.0, 111.7)
- removed the D4 at (270.0, 111.7)
- removed the D4 at (238.0, 111.7)
- removed the D4 at (206.0, 111.7)
- removed the D4 at (302.0, 94.7)
- removed the FIL15 at (288.5, 125.6)
- removed the FIL15 at (256.5, 91.6)
- removed the FIL15 at (224.5, 91.6)
- removed the FIL15 at (192.5, 91.6)
- removed the FIL15 at (288.5, 74.6)
- removed the FIL15 at (256.5, 74.6)
- removed the FIL15 at (224.5, 74.6)
- removed the FIL15 at (192.5, 74.6)
- removed the FIL15 at (288.5, 57.6)
- removed the FIL15 at (256.5, 57.6)
- removed the FIL15 at (224.5, 57.6)
- removed the FIL15 at (256.5, 125.6)
- removed the FIL15 at (224.5, 125.6)
- removed the FIL15 at (192.5, 125.6)
- removed the FIL15 at (288.5, 108.6)
- removed the FIL15 at (256.5, 108.6)
- removed the FIL15 at (224.5, 108.6)
- removed the FIL15 at (192.5, 108.6)
- removed the FIL15 at (288.5, 91.6)
- removed the FIL16 at (294.0, 125.6)
- removed the FIL16 at (262.0, 91.6)
- removed the FIL16 at (230.0, 91.6)
- removed the FIL16 at (198.0, 91.6)
- removed the FIL16 at (294.0, 74.6)
- removed the FIL16 at (262.0, 74.6)
- removed the FIL16 at (230.0, 74.6)
- removed the FIL16 at (198.0, 74.6)
- removed the FIL16 at (294.0, 57.6)
- removed the FIL16 at (262.0, 57.6)
- removed the FIL16 at (230.0, 57.6)
- removed the FIL16 at (262.0, 125.6)
- removed the FIL16 at (230.0, 125.6)
- removed the FIL16 at (198.0, 125.6)
- removed the FIL16 at (294.0, 108.6)
- removed the FIL16 at (262.0, 108.6)
- removed the FIL16 at (230.0, 108.6)
- removed the FIL16 at (198.0, 108.6)
- removed the FIL16 at (294.0, 91.6)
- removed the FIL17 at (283.0, 125.6)
- removed the FIL17 at (251.0, 91.6)
- removed the FIL17 at (219.0, 91.6)
- removed the FIL17 at (187.0, 91.6)
- removed the FIL17 at (283.0, 74.6)
- removed the FIL17 at (251.0, 74.6)
- removed the FIL17 at (219.0, 74.6)
- removed the FIL17 at (187.0, 74.6)
- removed the FIL17 at (283.0, 57.6)
- removed the FIL17 at (251.0, 57.6)
- removed the FIL17 at (219.0, 57.6)
- removed the FIL17 at (251.0, 125.6)
- removed the FIL17 at (219.0, 125.6)
- removed the FIL17 at (187.0, 125.6)
- removed the FIL17 at (283.0, 108.6)
- removed the FIL17 at (251.0, 108.6)
- removed the FIL17 at (219.0, 108.6)
- removed the FIL17 at (187.0, 108.6)
- removed the FIL17 at (283.0, 91.6)
- removed the J1 at (299.7, 123.7)
- removed the J1 at (267.7, 89.7)
- removed the J1 at (235.7, 89.7)
- removed the J1 at (203.7, 89.7)
- removed the J1 at (299.7, 72.7)
- removed the J1 at (267.7, 72.7)
- removed the J1 at (235.7, 72.7)
- removed the J1 at (203.7, 72.7)
- removed the J1 at (299.7, 55.7)
- removed the J1 at (267.7, 55.7)
- removed the J1 at (235.7, 55.7)
- removed the J1 at (267.7, 123.7)
- removed the J1 at (235.7, 123.7)
- removed the J1 at (203.7, 123.7)
- removed the J1 at (299.7, 106.7)
- removed the J1 at (267.7, 106.7)
- removed the J1 at (235.7, 106.7)
- removed the J1 at (203.7, 106.7)
- removed the J1 at (299.7, 89.7)
- removed the J2 at (302.4, 123.7)
- removed the J2 at (270.4, 89.7)
- removed the J2 at (238.4, 89.7)
- removed the J2 at (206.4, 89.7)
- removed the J2 at (302.4, 72.7)
- removed the J2 at (270.4, 72.7)
- removed the J2 at (238.4, 72.7)
- removed the J2 at (206.4, 72.7)
- removed the J2 at (302.4, 55.7)
- removed the J2 at (270.4, 55.7)
- removed the J2 at (238.4, 55.7)
- removed the J2 at (270.4, 123.7)
- removed the J2 at (238.4, 123.7)
- removed the J2 at (206.4, 123.7)
- removed the J2 at (302.4, 106.7)
- removed the J2 at (270.4, 106.7)
- removed the J2 at (238.4, 106.7)
- removed the J2 at (206.4, 106.7)
- removed the J2 at (302.4, 89.7)
- removed the J3 at (305.1, 123.7)
- removed the J3 at (273.1, 89.7)
- removed the J3 at (241.1, 89.7)
- removed the J3 at (209.1, 89.7)
- removed the J3 at (305.1, 72.7)
- removed the J3 at (273.1, 72.7)
- removed the J3 at (241.1, 72.7)
- removed the J3 at (209.1, 72.7)
- removed the J3 at (305.1, 55.7)
- removed the J3 at (273.1, 55.7)
- removed the J3 at (241.1, 55.7)
- removed the J3 at (273.1, 123.7)
- removed the J3 at (241.1, 123.7)
- removed the J3 at (209.1, 123.7)
- removed the J3 at (305.1, 106.7)
- removed the J3 at (273.1, 106.7)
- removed the J3 at (241.1, 106.7)
- removed the J3 at (209.1, 106.7)
- removed the J3 at (305.1, 89.7)
- removed the J4 at (307.3, 127.7)
- removed the J4 at (275.3, 93.7)
- removed the J4 at (243.3, 93.7)
- removed the J4 at (211.3, 93.7)
- removed the J4 at (307.3, 76.7)
- removed the J4 at (275.3, 76.7)
- removed the J4 at (243.3, 76.7)
- removed the J4 at (211.3, 76.7)
- removed the J4 at (307.3, 59.7)
- removed the J4 at (275.3, 59.7)
- removed the J4 at (243.3, 59.7)
- removed the J4 at (275.3, 127.7)
- removed the J4 at (243.3, 127.7)
- removed the J4 at (211.3, 127.7)
- removed the J4 at (307.3, 110.7)
- removed the J4 at (275.3, 110.7)
- removed the J4 at (243.3, 110.7)
- removed the J4 at (211.3, 110.7)
- removed the J4 at (307.3, 93.7)
- removed the J5 at (307.8, 123.7)
- removed the J5 at (275.8, 89.7)
- removed the J5 at (243.8, 89.7)
- removed the J5 at (211.8, 89.7)
- removed the J5 at (307.8, 72.7)
- removed the J5 at (275.8, 72.7)
- removed the J5 at (243.8, 72.7)
- removed the J5 at (211.8, 72.7)
- removed the J5 at (307.8, 55.7)
- removed the J5 at (275.8, 55.7)
- removed the J5 at (243.8, 55.7)
- removed the J5 at (275.8, 123.7)
- removed the J5 at (243.8, 123.7)
- removed the J5 at (211.8, 123.7)
- removed the J5 at (307.8, 106.7)
- removed the J5 at (275.8, 106.7)
- removed the J5 at (243.8, 106.7)
- removed the J5 at (211.8, 106.7)
- removed the J5 at (307.8, 89.7)
- removed the J6 at (307.3, 133.1)
- removed the J6 at (275.3, 99.1)
- removed the J6 at (243.3, 99.1)
- removed the J6 at (211.3, 99.1)
- removed the J6 at (307.3, 82.1)
- removed the J6 at (275.3, 82.1)
- removed the J6 at (243.3, 82.1)
- removed the J6 at (211.3, 82.1)
- removed the J6 at (307.3, 65.1)
- removed the J6 at (275.3, 65.1)
- removed the J6 at (243.3, 65.1)
- removed the J6 at (275.3, 133.1)
- removed the J6 at (243.3, 133.1)
- removed the J6 at (211.3, 133.1)
- removed the J6 at (307.3, 116.1)
- removed the J6 at (275.3, 116.1)
- removed the J6 at (243.3, 116.1)
- removed the J6 at (211.3, 116.1)
- removed the J6 at (307.3, 99.1)
- removed the J7 at (307.3, 135.8)
- removed the J7 at (275.3, 101.8)
- removed the J7 at (243.3, 101.8)
- removed the J7 at (211.3, 101.8)
- removed the J7 at (307.3, 84.8)
- removed the J7 at (275.3, 84.8)
- removed the J7 at (243.3, 84.8)
- removed the J7 at (211.3, 84.8)
- removed the J7 at (307.3, 67.8)
- removed the J7 at (275.3, 67.8)
- removed the J7 at (243.3, 67.8)
- removed the J7 at (275.3, 135.8)
- removed the J7 at (243.3, 135.8)
- removed the J7 at (211.3, 135.8)
- removed the J7 at (307.3, 118.8)
- removed the J7 at (275.3, 118.8)
- removed the J7 at (243.3, 118.8)
- removed the J7 at (211.3, 118.8)
- removed the J7 at (307.3, 101.8)
- removed the J8 at (307.3, 130.4)
- removed the J8 at (275.3, 96.4)
- removed the J8 at (243.3, 96.4)
- removed the J8 at (211.3, 96.4)
- removed the J8 at (307.3, 79.4)
- removed the J8 at (275.3, 79.4)
- removed the J8 at (243.3, 79.4)
- removed the J8 at (211.3, 79.4)
- removed the J8 at (307.3, 62.4)
- removed the J8 at (275.3, 62.4)
- removed the J8 at (243.3, 62.4)
- removed the J8 at (275.3, 130.4)
- removed the J8 at (243.3, 130.4)
- removed the J8 at (211.3, 130.4)
- removed the J8 at (307.3, 113.4)
- removed the J8 at (275.3, 113.4)
- removed the J8 at (243.3, 113.4)
- removed the J8 at (211.3, 113.4)
- removed the J8 at (307.3, 96.4)
- removed the J9 at (302.4, 135.4)
- removed the J9 at (270.4, 101.4)
- removed the J9 at (238.4, 101.4)
- removed the J9 at (206.4, 101.4)
- removed the J9 at (302.4, 84.4)
- removed the J9 at (270.4, 84.4)
- removed the J9 at (238.4, 84.4)
- removed the J9 at (206.4, 84.4)
- removed the J9 at (302.4, 67.4)
- removed the J9 at (270.4, 67.4)
- removed the J9 at (238.4, 67.4)
- removed the J9 at (270.4, 135.4)
- removed the J9 at (238.4, 135.4)
- removed the J9 at (206.4, 135.4)
- removed the J9 at (302.4, 118.4)
- removed the J9 at (270.4, 118.4)
- removed the J9 at (238.4, 118.4)
- removed the J9 at (206.4, 118.4)
- removed the J9 at (302.4, 101.4)
- removed the R37 at (298.1, 131.9)
- removed the R37 at (266.1, 97.9)
- removed the R37 at (234.1, 97.9)
- removed the R37 at (202.1, 97.9)
- removed the R37 at (298.1, 80.9)
- removed the R37 at (266.1, 80.9)
- removed the R37 at (234.1, 80.9)
- removed the R37 at (202.1, 80.9)
- removed the R37 at (298.1, 63.9)
- removed the R37 at (266.1, 63.9)
- removed the R37 at (234.1, 63.9)
- removed the R37 at (266.1, 131.9)
- removed the R37 at (234.1, 131.9)
- removed the R37 at (202.1, 131.9)
- removed the R37 at (298.1, 114.9)
- removed the R37 at (266.1, 114.9)
- removed the R37 at (234.1, 114.9)
- removed the R37 at (202.1, 114.9)
- removed the R37 at (298.1, 97.9)
- removed the R39 at (298.1, 135.7)
- removed the R39 at (266.1, 101.7)
- removed the R39 at (234.1, 101.7)
- removed the R39 at (202.1, 101.7)
- removed the R39 at (298.1, 84.7)
- removed the R39 at (266.1, 84.7)
- removed the R39 at (234.1, 84.7)
- removed the R39 at (202.1, 84.7)
- removed the R39 at (298.1, 67.7)
- removed the R39 at (266.1, 67.7)
- removed the R39 at (234.1, 67.7)
- removed the R39 at (266.1, 135.7)
- removed the R39 at (234.1, 135.7)
- removed the R39 at (202.1, 135.7)
- removed the R39 at (298.1, 118.7)
- removed the R39 at (266.1, 118.7)
- removed the R39 at (234.1, 118.7)
- removed the R39 at (202.1, 118.7)
- removed the R39 at (298.1, 101.7)
- removed the R40 at (298.1, 133.8)
- removed the R40 at (266.1, 99.8)
- removed the R40 at (234.1, 99.8)
- removed the R40 at (202.1, 99.8)
- removed the R40 at (298.1, 82.8)
- removed the R40 at (266.1, 82.8)
- removed the R40 at (234.1, 82.8)
- removed the R40 at (202.1, 82.8)
- removed the R40 at (298.1, 65.8)
- removed the R40 at (266.1, 65.8)
- removed the R40 at (234.1, 65.8)
- removed the R40 at (266.1, 133.8)
- removed the R40 at (234.1, 133.8)
- removed the R40 at (202.1, 133.8)
- removed the R40 at (298.1, 116.8)
- removed the R40 at (266.1, 116.8)
- removed the R40 at (234.1, 116.8)
- removed the R40 at (202.1, 116.8)
- removed the R40 at (298.1, 99.8)
- removed the mouse-bite-2mm-slot at (294.0, 121.0)
- removed the mouse-bite-2mm-slot at (262.0, 87.0)
- removed the mouse-bite-2mm-slot at (230.0, 87.0)
- removed the mouse-bite-2mm-slot at (198.0, 87.0)
- removed the mouse-bite-2mm-slot at (294.0, 70.0)
- removed the mouse-bite-2mm-slot at (262.0, 70.0)
- removed the mouse-bite-2mm-slot at (230.0, 70.0)
- removed the mouse-bite-2mm-slot at (278.0, 129.5)
- removed the mouse-bite-2mm-slot at (246.0, 129.5)
- removed the mouse-bite-2mm-slot at (214.0, 129.5)
- removed the mouse-bite-2mm-slot at (278.0, 112.5)
- removed the mouse-bite-2mm-slot at (262.0, 121.0)
- removed the mouse-bite-2mm-slot at (246.0, 112.5)
- removed the mouse-bite-2mm-slot at (214.0, 112.5)
- removed the mouse-bite-2mm-slot at (278.0, 95.5)
- removed the mouse-bite-2mm-slot at (246.0, 95.5)
- removed the mouse-bite-2mm-slot at (214.0, 95.5)
- removed the mouse-bite-2mm-slot at (278.0, 78.5)
- removed the mouse-bite-2mm-slot at (246.0, 78.5)
- removed the mouse-bite-2mm-slot at (214.0, 78.5)
- removed the mouse-bite-2mm-slot at (278.0, 61.5)
- removed the mouse-bite-2mm-slot at (246.0, 61.5)
- removed the mouse-bite-2mm-slot at (230.0, 121.0)
- removed the mouse-bite-2mm-slot at (214.0, 61.5)
- removed the mouse-bite-2mm-slot at (198.0, 70.0)
- removed the mouse-bite-2mm-slot at (198.0, 121.0)
- removed the mouse-bite-2mm-slot at (294.0, 104.0)
- removed the mouse-bite-2mm-slot at (262.0, 104.0)
- removed the mouse-bite-2mm-slot at (230.0, 104.0)
- removed the mouse-bite-2mm-slot at (198.0, 104.0)
- removed the mouse-bite-2mm-slot at (294.0, 87.0)
- added C64: 220μF, Capacitor_Tantalum_SMD:CP_EIA-7343-15_Kemet-W_Pad2.25x2.55mm_HandSolder, F.Cu at (73.1, 39.8)
- added C64: 220μF, Capacitor_Tantalum_SMD:CP_EIA-7343-15_Kemet-W_Pad2.25x2.55mm_HandSolder, F.Cu at (105.1, 73.8)
- added C64: 220μF, Capacitor_Tantalum_SMD:CP_EIA-7343-15_Kemet-W_Pad2.25x2.55mm_HandSolder, F.Cu at (137.1, 73.8)
- added C64: 220μF, Capacitor_Tantalum_SMD:CP_EIA-7343-15_Kemet-W_Pad2.25x2.55mm_HandSolder, F.Cu at (41.1, 90.8)
- added C64: 220μF, Capacitor_Tantalum_SMD:CP_EIA-7343-15_Kemet-W_Pad2.25x2.55mm_HandSolder, F.Cu at (73.1, 90.8)
- added C64: 220μF, Capacitor_Tantalum_SMD:CP_EIA-7343-15_Kemet-W_Pad2.25x2.55mm_HandSolder, F.Cu at (105.1, 90.8)
- added C64: 220μF, Capacitor_Tantalum_SMD:CP_EIA-7343-15_Kemet-W_Pad2.25x2.55mm_HandSolder, F.Cu at (137.1, 90.8)
- added C64: 220μF, Capacitor_Tantalum_SMD:CP_EIA-7343-15_Kemet-W_Pad2.25x2.55mm_HandSolder, F.Cu at (41.1, 107.8)
- added C64: 220μF, Capacitor_Tantalum_SMD:CP_EIA-7343-15_Kemet-W_Pad2.25x2.55mm_HandSolder, F.Cu at (73.1, 107.8)
- added C64: 220μF, Capacitor_Tantalum_SMD:CP_EIA-7343-15_Kemet-W_Pad2.25x2.55mm_HandSolder, F.Cu at (105.1, 107.8)
- added C64: 220μF, Capacitor_Tantalum_SMD:CP_EIA-7343-15_Kemet-W_Pad2.25x2.55mm_HandSolder, F.Cu at (137.1, 107.8)
- added C64: 220μF, Capacitor_Tantalum_SMD:CP_EIA-7343-15_Kemet-W_Pad2.25x2.55mm_HandSolder, F.Cu at (105.1, 39.8)
- added C64: 220μF, Capacitor_Tantalum_SMD:CP_EIA-7343-15_Kemet-W_Pad2.25x2.55mm_HandSolder, F.Cu at (137.1, 39.8)
- added C64: 220μF, Capacitor_Tantalum_SMD:CP_EIA-7343-15_Kemet-W_Pad2.25x2.55mm_HandSolder, F.Cu at (41.1, 56.8)
- added C64: 220μF, Capacitor_Tantalum_SMD:CP_EIA-7343-15_Kemet-W_Pad2.25x2.55mm_HandSolder, F.Cu at (73.1, 56.8)
- added C64: 220μF, Capacitor_Tantalum_SMD:CP_EIA-7343-15_Kemet-W_Pad2.25x2.55mm_HandSolder, F.Cu at (105.1, 56.8)
- added C64: 220μF, Capacitor_Tantalum_SMD:CP_EIA-7343-15_Kemet-W_Pad2.25x2.55mm_HandSolder, F.Cu at (137.1, 56.8)
- added C64: 220μF, Capacitor_Tantalum_SMD:CP_EIA-7343-15_Kemet-W_Pad2.25x2.55mm_HandSolder, F.Cu at (41.1, 73.8)
- added C64: 220μF, Capacitor_Tantalum_SMD:CP_EIA-7343-15_Kemet-W_Pad2.25x2.55mm_HandSolder, F.Cu at (73.1, 73.8)
- added C66: 50pF, Capacitor_SMD:C_0603_1608Metric_Pad1.05x0.95mm_HandSolder, F.Cu at (68.5, 31.8)
- added C66: 50pF, Capacitor_SMD:C_0603_1608Metric_Pad1.05x0.95mm_HandSolder, F.Cu at (100.5, 65.8)
- added C66: 50pF, Capacitor_SMD:C_0603_1608Metric_Pad1.05x0.95mm_HandSolder, F.Cu at (132.5, 65.8)
- added C66: 50pF, Capacitor_SMD:C_0603_1608Metric_Pad1.05x0.95mm_HandSolder, F.Cu at (36.5, 82.8)
- added C66: 50pF, Capacitor_SMD:C_0603_1608Metric_Pad1.05x0.95mm_HandSolder, F.Cu at (68.5, 82.8)
- added C66: 50pF, Capacitor_SMD:C_0603_1608Metric_Pad1.05x0.95mm_HandSolder, F.Cu at (100.5, 82.8)
- added C66: 50pF, Capacitor_SMD:C_0603_1608Metric_Pad1.05x0.95mm_HandSolder, F.Cu at (132.5, 82.8)
- added C66: 50pF, Capacitor_SMD:C_0603_1608Metric_Pad1.05x0.95mm_HandSolder, F.Cu at (36.5, 99.8)
- added C66: 50pF, Capacitor_SMD:C_0603_1608Metric_Pad1.05x0.95mm_HandSolder, F.Cu at (68.5, 99.8)
- added C66: 50pF, Capacitor_SMD:C_0603_1608Metric_Pad1.05x0.95mm_HandSolder, F.Cu at (100.5, 99.8)
- added C66: 50pF, Capacitor_SMD:C_0603_1608Metric_Pad1.05x0.95mm_HandSolder, F.Cu at (132.5, 99.8)
- added C66: 50pF, Capacitor_SMD:C_0603_1608Metric_Pad1.05x0.95mm_HandSolder, F.Cu at (100.5, 31.8)
- added C66: 50pF, Capacitor_SMD:C_0603_1608Metric_Pad1.05x0.95mm_HandSolder, F.Cu at (132.5, 31.8)
- added C66: 50pF, Capacitor_SMD:C_0603_1608Metric_Pad1.05x0.95mm_HandSolder, F.Cu at (36.5, 48.8)
- added C66: 50pF, Capacitor_SMD:C_0603_1608Metric_Pad1.05x0.95mm_HandSolder, F.Cu at (68.5, 48.8)
- added C66: 50pF, Capacitor_SMD:C_0603_1608Metric_Pad1.05x0.95mm_HandSolder, F.Cu at (100.5, 48.8)
- added C66: 50pF, Capacitor_SMD:C_0603_1608Metric_Pad1.05x0.95mm_HandSolder, F.Cu at (132.5, 48.8)
- added C66: 50pF, Capacitor_SMD:C_0603_1608Metric_Pad1.05x0.95mm_HandSolder, F.Cu at (36.5, 65.8)
- added C66: 50pF, Capacitor_SMD:C_0603_1608Metric_Pad1.05x0.95mm_HandSolder, F.Cu at (68.5, 65.8)
- added C69: 220μF, Capacitor_Tantalum_SMD:CP_EIA-7343-15_Kemet-W_Pad2.25x2.55mm_HandSolder, F.Cu at (67.6, 73.8)
- added C69: 220μF, Capacitor_Tantalum_SMD:CP_EIA-7343-15_Kemet-W_Pad2.25x2.55mm_HandSolder, F.Cu at (99.6, 73.8)
- added C69: 220μF, Capacitor_Tantalum_SMD:CP_EIA-7343-15_Kemet-W_Pad2.25x2.55mm_HandSolder, F.Cu at (131.6, 73.8)
- added C69: 220μF, Capacitor_Tantalum_SMD:CP_EIA-7343-15_Kemet-W_Pad2.25x2.55mm_HandSolder, F.Cu at (35.6, 90.8)
- added C69: 220μF, Capacitor_Tantalum_SMD:CP_EIA-7343-15_Kemet-W_Pad2.25x2.55mm_HandSolder, F.Cu at (67.6, 90.8)
- added C69: 220μF, Capacitor_Tantalum_SMD:CP_EIA-7343-15_Kemet-W_Pad2.25x2.55mm_HandSolder, F.Cu at (99.6, 90.8)
- added C69: 220μF, Capacitor_Tantalum_SMD:CP_EIA-7343-15_Kemet-W_Pad2.25x2.55mm_HandSolder, F.Cu at (131.6, 90.8)
- added C69: 220μF, Capacitor_Tantalum_SMD:CP_EIA-7343-15_Kemet-W_Pad2.25x2.55mm_HandSolder, F.Cu at (35.6, 107.8)
- added C69: 220μF, Capacitor_Tantalum_SMD:CP_EIA-7343-15_Kemet-W_Pad2.25x2.55mm_HandSolder, F.Cu at (67.6, 107.8)
- added C69: 220μF, Capacitor_Tantalum_SMD:CP_EIA-7343-15_Kemet-W_Pad2.25x2.55mm_HandSolder, F.Cu at (99.6, 107.8)
- added C69: 220μF, Capacitor_Tantalum_SMD:CP_EIA-7343-15_Kemet-W_Pad2.25x2.55mm_HandSolder, F.Cu at (67.6, 39.8)
- added C69: 220μF, Capacitor_Tantalum_SMD:CP_EIA-7343-15_Kemet-W_Pad2.25x2.55mm_HandSolder, F.Cu at (131.6, 107.8)
- added C69: 220μF, Capacitor_Tantalum_SMD:CP_EIA-7343-15_Kemet-W_Pad2.25x2.55mm_HandSolder, F.Cu at (99.6, 39.8)
- added C69: 220μF, Capacitor_Tantalum_SMD:CP_EIA-7343-15_Kemet-W_Pad2.25x2.55mm_HandSolder, F.Cu at (131.6, 39.8)
- added C69: 220μF, Capacitor_Tantalum_SMD:CP_EIA-7343-15_Kemet-W_Pad2.25x2.55mm_HandSolder, F.Cu at (35.6, 56.8)
- added C69: 220μF, Capacitor_Tantalum_SMD:CP_EIA-7343-15_Kemet-W_Pad2.25x2.55mm_HandSolder, F.Cu at (67.6, 56.8)
- added C69: 220μF, Capacitor_Tantalum_SMD:CP_EIA-7343-15_Kemet-W_Pad2.25x2.55mm_HandSolder, F.Cu at (99.6, 56.8)
- added C69: 220μF, Capacitor_Tantalum_SMD:CP_EIA-7343-15_Kemet-W_Pad2.25x2.55mm_HandSolder, F.Cu at (131.6, 56.8)
- added C69: 220μF, Capacitor_Tantalum_SMD:CP_EIA-7343-15_Kemet-W_Pad2.25x2.55mm_HandSolder, F.Cu at (35.6, 73.8)
- added C72: 100pF, Capacitor_SMD:C_0603_1608Metric_Pad1.05x0.95mm_HandSolder, F.Cu at (65.9, 32.7)
- added C72: 100pF, Capacitor_SMD:C_0603_1608Metric_Pad1.05x0.95mm_HandSolder, F.Cu at (97.9, 66.7)
- added C72: 100pF, Capacitor_SMD:C_0603_1608Metric_Pad1.05x0.95mm_HandSolder, F.Cu at (129.9, 66.7)
- added C72: 100pF, Capacitor_SMD:C_0603_1608Metric_Pad1.05x0.95mm_HandSolder, F.Cu at (33.9, 83.7)
- added C72: 100pF, Capacitor_SMD:C_0603_1608Metric_Pad1.05x0.95mm_HandSolder, F.Cu at (65.9, 83.7)
- added C72: 100pF, Capacitor_SMD:C_0603_1608Metric_Pad1.05x0.95mm_HandSolder, F.Cu at (97.9, 83.7)
- added C72: 100pF, Capacitor_SMD:C_0603_1608Metric_Pad1.05x0.95mm_HandSolder, F.Cu at (129.9, 83.7)
- added C72: 100pF, Capacitor_SMD:C_0603_1608Metric_Pad1.05x0.95mm_HandSolder, F.Cu at (33.9, 100.7)
- added C72: 100pF, Capacitor_SMD:C_0603_1608Metric_Pad1.05x0.95mm_HandSolder, F.Cu at (65.9, 100.7)
- added C72: 100pF, Capacitor_SMD:C_0603_1608Metric_Pad1.05x0.95mm_HandSolder, F.Cu at (97.9, 100.7)
- added C72: 100pF, Capacitor_SMD:C_0603_1608Metric_Pad1.05x0.95mm_HandSolder, F.Cu at (129.9, 100.7)
- added C72: 100pF, Capacitor_SMD:C_0603_1608Metric_Pad1.05x0.95mm_HandSolder, F.Cu at (97.9, 32.7)
- added C72: 100pF, Capacitor_SMD:C_0603_1608Metric_Pad1.05x0.95mm_HandSolder, F.Cu at (129.9, 32.7)
- added C72: 100pF, Capacitor_SMD:C_0603_1608Metric_Pad1.05x0.95mm_HandSolder, F.Cu at (33.9, 49.7)
- added C72: 100pF, Capacitor_SMD:C_0603_1608Metric_Pad1.05x0.95mm_HandSolder, F.Cu at (65.9, 49.7)
- added C72: 100pF, Capacitor_SMD:C_0603_1608Metric_Pad1.05x0.95mm_HandSolder, F.Cu at (97.9, 49.7)
- added C72: 100pF, Capacitor_SMD:C_0603_1608Metric_Pad1.05x0.95mm_HandSolder, F.Cu at (129.9, 49.7)
- added C72: 100pF, Capacitor_SMD:C_0603_1608Metric_Pad1.05x0.95mm_HandSolder, F.Cu at (33.9, 66.7)
- added C72: 100pF, Capacitor_SMD:C_0603_1608Metric_Pad1.05x0.95mm_HandSolder, F.Cu at (65.9, 66.7)
- added C74: 50pF, Capacitor_SMD:C_0603_1608Metric_Pad1.05x0.95mm_HandSolder, F.Cu at (74.0, 31.8)
- added C74: 50pF, Capacitor_SMD:C_0603_1608Metric_Pad1.05x0.95mm_HandSolder, F.Cu at (106.0, 65.8)
- added C74: 50pF, Capacitor_SMD:C_0603_1608Metric_Pad1.05x0.95mm_HandSolder, F.Cu at (138.0, 65.8)
- added C74: 50pF, Capacitor_SMD:C_0603_1608Metric_Pad1.05x0.95mm_HandSolder, F.Cu at (42.0, 82.8)
- added C74: 50pF, Capacitor_SMD:C_0603_1608Metric_Pad1.05x0.95mm_HandSolder, F.Cu at (74.0, 82.8)
- added C74: 50pF, Capacitor_SMD:C_0603_1608Metric_Pad1.05x0.95mm_HandSolder, F.Cu at (106.0, 82.8)
- added C74: 50pF, Capacitor_SMD:C_0603_1608Metric_Pad1.05x0.95mm_HandSolder, F.Cu at (138.0, 82.8)
- added C74: 50pF, Capacitor_SMD:C_0603_1608Metric_Pad1.05x0.95mm_HandSolder, F.Cu at (42.0, 99.8)
- added C74: 50pF, Capacitor_SMD:C_0603_1608Metric_Pad1.05x0.95mm_HandSolder, F.Cu at (74.0, 99.8)
- added C74: 50pF, Capacitor_SMD:C_0603_1608Metric_Pad1.05x0.95mm_HandSolder, F.Cu at (106.0, 99.8)
- added C74: 50pF, Capacitor_SMD:C_0603_1608Metric_Pad1.05x0.95mm_HandSolder, F.Cu at (138.0, 99.8)
- added C74: 50pF, Capacitor_SMD:C_0603_1608Metric_Pad1.05x0.95mm_HandSolder, F.Cu at (106.0, 31.8)
- added C74: 50pF, Capacitor_SMD:C_0603_1608Metric_Pad1.05x0.95mm_HandSolder, F.Cu at (138.0, 31.8)
- added C74: 50pF, Capacitor_SMD:C_0603_1608Metric_Pad1.05x0.95mm_HandSolder, F.Cu at (42.0, 48.8)
- added C74: 50pF, Capacitor_SMD:C_0603_1608Metric_Pad1.05x0.95mm_HandSolder, F.Cu at (74.0, 48.8)
- added C74: 50pF, Capacitor_SMD:C_0603_1608Metric_Pad1.05x0.95mm_HandSolder, F.Cu at (106.0, 48.8)
- added C74: 50pF, Capacitor_SMD:C_0603_1608Metric_Pad1.05x0.95mm_HandSolder, F.Cu at (138.0, 48.8)
- added C74: 50pF, Capacitor_SMD:C_0603_1608Metric_Pad1.05x0.95mm_HandSolder, F.Cu at (42.0, 65.8)
- added C74: 50pF, Capacitor_SMD:C_0603_1608Metric_Pad1.05x0.95mm_HandSolder, F.Cu at (74.0, 65.8)
- added C78: 100pF, Capacitor_SMD:C_0603_1608Metric_Pad1.05x0.95mm_HandSolder, F.Cu at (71.4, 32.7)
- added C78: 100pF, Capacitor_SMD:C_0603_1608Metric_Pad1.05x0.95mm_HandSolder, F.Cu at (103.4, 66.7)
- added C78: 100pF, Capacitor_SMD:C_0603_1608Metric_Pad1.05x0.95mm_HandSolder, F.Cu at (135.4, 66.7)
- added C78: 100pF, Capacitor_SMD:C_0603_1608Metric_Pad1.05x0.95mm_HandSolder, F.Cu at (39.4, 83.7)
- added C78: 100pF, Capacitor_SMD:C_0603_1608Metric_Pad1.05x0.95mm_HandSolder, F.Cu at (71.4, 83.7)
- added C78: 100pF, Capacitor_SMD:C_0603_1608Metric_Pad1.05x0.95mm_HandSolder, F.Cu at (103.4, 83.7)
- added C78: 100pF, Capacitor_SMD:C_0603_1608Metric_Pad1.05x0.95mm_HandSolder, F.Cu at (135.4, 83.7)
- added C78: 100pF, Capacitor_SMD:C_0603_1608Metric_Pad1.05x0.95mm_HandSolder, F.Cu at (39.4, 100.7)
- added C78: 100pF, Capacitor_SMD:C_0603_1608Metric_Pad1.05x0.95mm_HandSolder, F.Cu at (71.4, 100.7)
- added C78: 100pF, Capacitor_SMD:C_0603_1608Metric_Pad1.05x0.95mm_HandSolder, F.Cu at (103.4, 100.7)
- added C78: 100pF, Capacitor_SMD:C_0603_1608Metric_Pad1.05x0.95mm_HandSolder, F.Cu at (135.4, 100.7)
- added C78: 100pF, Capacitor_SMD:C_0603_1608Metric_Pad1.05x0.95mm_HandSolder, F.Cu at (103.4, 32.7)
- added C78: 100pF, Capacitor_SMD:C_0603_1608Metric_Pad1.05x0.95mm_HandSolder, F.Cu at (135.4, 32.7)
- added C78: 100pF, Capacitor_SMD:C_0603_1608Metric_Pad1.05x0.95mm_HandSolder, F.Cu at (39.4, 49.7)
- added C78: 100pF, Capacitor_SMD:C_0603_1608Metric_Pad1.05x0.95mm_HandSolder, F.Cu at (71.4, 49.7)
- added C78: 100pF, Capacitor_SMD:C_0603_1608Metric_Pad1.05x0.95mm_HandSolder, F.Cu at (103.4, 49.7)
- added C78: 100pF, Capacitor_SMD:C_0603_1608Metric_Pad1.05x0.95mm_HandSolder, F.Cu at (135.4, 49.7)
- added C78: 100pF, Capacitor_SMD:C_0603_1608Metric_Pad1.05x0.95mm_HandSolder, F.Cu at (39.4, 66.7)
- added C78: 100pF, Capacitor_SMD:C_0603_1608Metric_Pad1.05x0.95mm_HandSolder, F.Cu at (71.4, 66.7)
- added C83: 50pF, Capacitor_SMD:C_0603_1608Metric_Pad1.05x0.95mm_HandSolder, F.Cu at (63.0, 31.8)
- added C83: 50pF, Capacitor_SMD:C_0603_1608Metric_Pad1.05x0.95mm_HandSolder, F.Cu at (95.0, 65.8)
- added C83: 50pF, Capacitor_SMD:C_0603_1608Metric_Pad1.05x0.95mm_HandSolder, F.Cu at (127.0, 65.8)
- added C83: 50pF, Capacitor_SMD:C_0603_1608Metric_Pad1.05x0.95mm_HandSolder, F.Cu at (31.0, 82.8)
- added C83: 50pF, Capacitor_SMD:C_0603_1608Metric_Pad1.05x0.95mm_HandSolder, F.Cu at (63.0, 82.8)
- added C83: 50pF, Capacitor_SMD:C_0603_1608Metric_Pad1.05x0.95mm_HandSolder, F.Cu at (95.0, 82.8)
- added C83: 50pF, Capacitor_SMD:C_0603_1608Metric_Pad1.05x0.95mm_HandSolder, F.Cu at (127.0, 82.8)
- added C83: 50pF, Capacitor_SMD:C_0603_1608Metric_Pad1.05x0.95mm_HandSolder, F.Cu at (31.0, 99.8)
- added C83: 50pF, Capacitor_SMD:C_0603_1608Metric_Pad1.05x0.95mm_HandSolder, F.Cu at (63.0, 99.8)
- added C83: 50pF, Capacitor_SMD:C_0603_1608Metric_Pad1.05x0.95mm_HandSolder, F.Cu at (95.0, 99.8)
- added C83: 50pF, Capacitor_SMD:C_0603_1608Metric_Pad1.05x0.95mm_HandSolder, F.Cu at (127.0, 99.8)
- added C83: 50pF, Capacitor_SMD:C_0603_1608Metric_Pad1.05x0.95mm_HandSolder, F.Cu at (95.0, 31.8)
- added C83: 50pF, Capacitor_SMD:C_0603_1608Metric_Pad1.05x0.95mm_HandSolder, F.Cu at (127.0, 31.8)
- added C83: 50pF, Capacitor_SMD:C_0603_1608Metric_Pad1.05x0.95mm_HandSolder, F.Cu at (31.0, 48.8)
- added C83: 50pF, Capacitor_SMD:C_0603_1608Metric_Pad1.05x0.95mm_HandSolder, F.Cu at (63.0, 48.8)
- added C83: 50pF, Capacitor_SMD:C_0603_1608Metric_Pad1.05x0.95mm_HandSolder, F.Cu at (95.0, 48.8)
- added C83: 50pF, Capacitor_SMD:C_0603_1608Metric_Pad1.05x0.95mm_HandSolder, F.Cu at (127.0, 48.8)
- added C83: 50pF, Capacitor_SMD:C_0603_1608Metric_Pad1.05x0.95mm_HandSolder, F.Cu at (31.0, 65.8)
- added C83: 50pF, Capacitor_SMD:C_0603_1608Metric_Pad1.05x0.95mm_HandSolder, F.Cu at (63.0, 65.8)
- added C84: 220μF, Capacitor_Tantalum_SMD:CP_EIA-7343-15_Kemet-W_Pad2.25x2.55mm_HandSolder, F.Cu at (62.1, 73.8)
- added C84: 220μF, Capacitor_Tantalum_SMD:CP_EIA-7343-15_Kemet-W_Pad2.25x2.55mm_HandSolder, F.Cu at (94.1, 73.8)
- added C84: 220μF, Capacitor_Tantalum_SMD:CP_EIA-7343-15_Kemet-W_Pad2.25x2.55mm_HandSolder, F.Cu at (126.1, 73.8)
- added C84: 220μF, Capacitor_Tantalum_SMD:CP_EIA-7343-15_Kemet-W_Pad2.25x2.55mm_HandSolder, F.Cu at (30.1, 90.8)
- added C84: 220μF, Capacitor_Tantalum_SMD:CP_EIA-7343-15_Kemet-W_Pad2.25x2.55mm_HandSolder, F.Cu at (62.1, 90.8)
- added C84: 220μF, Capacitor_Tantalum_SMD:CP_EIA-7343-15_Kemet-W_Pad2.25x2.55mm_HandSolder, F.Cu at (94.1, 90.8)
- added C84: 220μF, Capacitor_Tantalum_SMD:CP_EIA-7343-15_Kemet-W_Pad2.25x2.55mm_HandSolder, F.Cu at (126.1, 90.8)
- added C84: 220μF, Capacitor_Tantalum_SMD:CP_EIA-7343-15_Kemet-W_Pad2.25x2.55mm_HandSolder, F.Cu at (30.1, 107.8)
- added C84: 220μF, Capacitor_Tantalum_SMD:CP_EIA-7343-15_Kemet-W_Pad2.25x2.55mm_HandSolder, F.Cu at (62.1, 107.8)
- added C84: 220μF, Capacitor_Tantalum_SMD:CP_EIA-7343-15_Kemet-W_Pad2.25x2.55mm_HandSolder, F.Cu at (94.1, 107.8)
- added C84: 220μF, Capacitor_Tantalum_SMD:CP_EIA-7343-15_Kemet-W_Pad2.25x2.55mm_HandSolder, F.Cu at (62.1, 39.8)
- added C84: 220μF, Capacitor_Tantalum_SMD:CP_EIA-7343-15_Kemet-W_Pad2.25x2.55mm_HandSolder, F.Cu at (126.1, 107.8)
- added C84: 220μF, Capacitor_Tantalum_SMD:CP_EIA-7343-15_Kemet-W_Pad2.25x2.55mm_HandSolder, F.Cu at (94.1, 39.8)
- added C84: 220μF, Capacitor_Tantalum_SMD:CP_EIA-7343-15_Kemet-W_Pad2.25x2.55mm_HandSolder, F.Cu at (126.1, 39.8)
- added C84: 220μF, Capacitor_Tantalum_SMD:CP_EIA-7343-15_Kemet-W_Pad2.25x2.55mm_HandSolder, F.Cu at (30.1, 56.8)
- added C84: 220μF, Capacitor_Tantalum_SMD:CP_EIA-7343-15_Kemet-W_Pad2.25x2.55mm_HandSolder, F.Cu at (62.1, 56.8)
- added C84: 220μF, Capacitor_Tantalum_SMD:CP_EIA-7343-15_Kemet-W_Pad2.25x2.55mm_HandSolder, F.Cu at (94.1, 56.8)
- added C84: 220μF, Capacitor_Tantalum_SMD:CP_EIA-7343-15_Kemet-W_Pad2.25x2.55mm_HandSolder, F.Cu at (126.1, 56.8)
- added C84: 220μF, Capacitor_Tantalum_SMD:CP_EIA-7343-15_Kemet-W_Pad2.25x2.55mm_HandSolder, F.Cu at (30.1, 73.8)
- added C85: 100pF, Capacitor_SMD:C_0603_1608Metric_Pad1.05x0.95mm_HandSolder, F.Cu at (60.4, 32.7)
- added C85: 100pF, Capacitor_SMD:C_0603_1608Metric_Pad1.05x0.95mm_HandSolder, F.Cu at (92.4, 66.7)
- added C85: 100pF, Capacitor_SMD:C_0603_1608Metric_Pad1.05x0.95mm_HandSolder, F.Cu at (124.4, 66.7)
- added C85: 100pF, Capacitor_SMD:C_0603_1608Metric_Pad1.05x0.95mm_HandSolder, F.Cu at (28.4, 83.7)
- added C85: 100pF, Capacitor_SMD:C_0603_1608Metric_Pad1.05x0.95mm_HandSolder, F.Cu at (60.4, 83.7)
- added C85: 100pF, Capacitor_SMD:C_0603_1608Metric_Pad1.05x0.95mm_HandSolder, F.Cu at (92.4, 83.7)
- added C85: 100pF, Capacitor_SMD:C_0603_1608Metric_Pad1.05x0.95mm_HandSolder, F.Cu at (124.4, 83.7)
- added C85: 100pF, Capacitor_SMD:C_0603_1608Metric_Pad1.05x0.95mm_HandSolder, F.Cu at (28.4, 100.7)
- added C85: 100pF, Capacitor_SMD:C_0603_1608Metric_Pad1.05x0.95mm_HandSolder, F.Cu at (60.4, 100.7)
- added C85: 100pF, Capacitor_SMD:C_0603_1608Metric_Pad1.05x0.95mm_HandSolder, F.Cu at (92.4, 100.7)
- added C85: 100pF, Capacitor_SMD:C_0603_1608Metric_Pad1.05x0.95mm_HandSolder, F.Cu at (124.4, 100.7)
- added C85: 100pF, Capacitor_SMD:C_0603_1608Metric_Pad1.05x0.95mm_HandSolder, F.Cu at (92.4, 32.7)
- added C85: 100pF, Capacitor_SMD:C_0603_1608Metric_Pad1.05x0.95mm_HandSolder, F.Cu at (124.4, 32.7)
- added C85: 100pF, Capacitor_SMD:C_0603_1608Metric_Pad1.05x0.95mm_HandSolder, F.Cu at (28.4, 49.7)
- added C85: 100pF, Capacitor_SMD:C_0603_1608Metric_Pad1.05x0.95mm_HandSolder, F.Cu at (60.4, 49.7)
- added C85: 100pF, Capacitor_SMD:C_0603_1608Metric_Pad1.05x0.95mm_HandSolder, F.Cu at (92.4, 49.7)
- added C85: 100pF, Capacitor_SMD:C_0603_1608Metric_Pad1.05x0.95mm_HandSolder, F.Cu at (124.4, 49.7)
- added C85: 100pF, Capacitor_SMD:C_0603_1608Metric_Pad1.05x0.95mm_HandSolder, F.Cu at (28.4, 66.7)
- added C85: 100pF, Capacitor_SMD:C_0603_1608Metric_Pad1.05x0.95mm_HandSolder, F.Cu at (60.4, 66.7)
- added D1: PESD5V0U1BA, Diode_SMD:D_SOD-323_HandSoldering, F.Cu at (141.4, 66.4)
- added D1: PESD5V0U1BA, Diode_SMD:D_SOD-323_HandSoldering, F.Cu at (109.4, 66.4)
- added D1: PESD5V0U1BA, Diode_SMD:D_SOD-323_HandSoldering, F.Cu at (77.4, 66.4)
- added D1: PESD5V0U1BA, Diode_SMD:D_SOD-323_HandSoldering, F.Cu at (77.4, 32.4)
- added D1: PESD5V0U1BA, Diode_SMD:D_SOD-323_HandSoldering, F.Cu at (109.4, 32.4)
- added D1: PESD5V0U1BA, Diode_SMD:D_SOD-323_HandSoldering, F.Cu at (141.4, 32.4)
- added D1: PESD5V0U1BA, Diode_SMD:D_SOD-323_HandSoldering, F.Cu at (45.4, 49.4)
- added D1: PESD5V0U1BA, Diode_SMD:D_SOD-323_HandSoldering, F.Cu at (77.4, 49.4)
- added D1: PESD5V0U1BA, Diode_SMD:D_SOD-323_HandSoldering, F.Cu at (109.4, 49.4)
- added D1: PESD5V0U1BA, Diode_SMD:D_SOD-323_HandSoldering, F.Cu at (141.4, 49.4)
- added D1: PESD5V0U1BA, Diode_SMD:D_SOD-323_HandSoldering, F.Cu at (109.4, 100.4)
- added D1: PESD5V0U1BA, Diode_SMD:D_SOD-323_HandSoldering, F.Cu at (45.4, 66.4)
- added D1: PESD5V0U1BA, Diode_SMD:D_SOD-323_HandSoldering, F.Cu at (141.4, 100.4)
- added D1: PESD5V0U1BA, Diode_SMD:D_SOD-323_HandSoldering, F.Cu at (77.4, 100.4)
- added D1: PESD5V0U1BA, Diode_SMD:D_SOD-323_HandSoldering, F.Cu at (45.4, 100.4)
- added D1: PESD5V0U1BA, Diode_SMD:D_SOD-323_HandSoldering, F.Cu at (141.4, 83.4)
- added D1: PESD5V0U1BA, Diode_SMD:D_SOD-323_HandSoldering, F.Cu at (77.4, 83.4)
- added D1: PESD5V0U1BA, Diode_SMD:D_SOD-323_HandSoldering, F.Cu at (109.4, 83.4)
- added D1: PESD5V0U1BA, Diode_SMD:D_SOD-323_HandSoldering, F.Cu at (45.4, 83.4)
- added D2: PESD5V0U1BA, Diode_SMD:D_SOD-323_HandSoldering, F.Cu at (77.4, 53.7)
- added D2: PESD5V0U1BA, Diode_SMD:D_SOD-323_HandSoldering, F.Cu at (109.4, 53.7)
- added D2: PESD5V0U1BA, Diode_SMD:D_SOD-323_HandSoldering, F.Cu at (141.4, 53.7)
- added D2: PESD5V0U1BA, Diode_SMD:D_SOD-323_HandSoldering, F.Cu at (45.4, 70.7)
- added D2: PESD5V0U1BA, Diode_SMD:D_SOD-323_HandSoldering, F.Cu at (77.4, 70.7)
- added D2: PESD5V0U1BA, Diode_SMD:D_SOD-323_HandSoldering, F.Cu at (109.4, 70.7)
- added D2: PESD5V0U1BA, Diode_SMD:D_SOD-323_HandSoldering, F.Cu at (141.4, 70.7)
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Other:
- board size 126 x 83 mm -> 126 x 95 mm
- board text added: "Don’t forget to visit consolebytes.com Blahhh!!!"
- board text added: "Wii are one. Wii are many."
- board text added: "by Job#3556 and Commandblock6417"
- board text added: "consolebytes.com/minirgbii"
- board text added: "miniRGBii PiiCiiBii panel 4x5"
- board text removed: "consolebytes.com/index.php/ community/postid/37/"
